File: XG_Mobile_Dock.kicad_pcb (KiCad board)
At the start: 2 copper layers, 172.2 x 76.7 mm, 14 parts

Commit message: Updated schematics
Parts:
- removed the REF** at (144.8, 71.1)
- added C1: 47µF, Capacitor_Tantalum_SMD:CP_EIA-7343-43_Kemet-X, F.Cu at (-62.6, 5.92)
- added C10: 0.1µF, Capacitor_SMD:C_0402_1005Metric, F.Cu at (-32.4, 26.4)
- added C11: 0.1µF, Capacitor_SMD:C_0402_1005Metric, F.Cu at (-32.4, 28.4)
- added C12: 0.1µF, Capacitor_SMD:C_0402_1005Metric, F.Cu at (-32.4, 30.3)
- added C13: 0.1µF, Capacitor_SMD:C_0402_1005Metric, F.Cu at (-32.4, 32.3)
- added C14: 0.1µF, Capacitor_SMD:C_0402_1005Metric, F.Cu at (-32.4, 34.3)
- added C15: 0.01µF, Capacitor_SMD:C_0402_1005Metric, F.Cu at (-32.4, 36.3)
- added C16: 0.1µF, Capacitor_SMD:C_0402_1005Metric, F.Cu at (-32.4, 38.2)
- added C17: 0.1µF, Capacitor_SMD:C_0402_1005Metric, F.Cu at (-29.5, 26.4)
- added C18: 220pF, Capacitor_SMD:C_0201_0603Metric, F.Cu at (-37.6, 24.3)
- added C19: 0.01µF, Capacitor_SMD:C_0402_1005Metric, F.Cu at (-29.5, 28.4)
- added C2: 47µF, Capacitor_Tantalum_SMD:CP_EIA-7343-43_Kemet-X, F.Cu at (-62.6, 11.8)
- added C20: 0.1µF, Capacitor_SMD:C_0402_1005Metric, F.Cu at (-47.6, 25.5)
- added C21: 1µF, Capacitor_SMD:C_0603_1608Metric, F.Cu at (-55.6, 15.9)
- added C22: 10µF, Capacitor_SMD:C_0402_1005Metric, F.Cu at (-44.7, 15.7)
- added C23: 10µF, Capacitor_SMD:C_0402_1005Metric, F.Cu at (-44.7, 17.6)
- added C24: 10µF, Capacitor_SMD:C_0402_1005Metric, F.Cu at (-44.7, 19.6)
- added C25: 10µF, Capacitor_SMD:C_0402_1005Metric, F.Cu at (-44.7, 21.6)
- added C26: 10µF, Capacitor_SMD:C_0402_1005Metric, F.Cu at (-44.7, 23.6)
- added C27: 0.1µF, Capacitor_SMD:C_0402_1005Metric, F.Cu at (-29.5, 30.3)
- added C28: 0.1µF, Capacitor_SMD:C_0402_1005Metric, F.Cu at (-29.5, 32.3)
- added C29: 0.1µF, Capacitor_SMD:C_0402_1005Metric, F.Cu at (-29.5, 34.3)
- added C3: 22µF, Capacitor_SMD:C_0805_2012Metric, F.Cu at (-51.4, 31.0)
- added C30: 0.1µF, Capacitor_SMD:C_0402_1005Metric, F.Cu at (-29.5, 36.3)
- added C31: 0.1µF, Capacitor_SMD:C_0402_1005Metric, F.Cu at (-29.5, 38.2)
- added C32: 0.01µF, Capacitor_SMD:C_0402_1005Metric, F.Cu at (-26.6, 26.4)
- added C33: 0.1µF, Capacitor_SMD:C_0402_1005Metric, F.Cu at (-26.6, 28.4)
- added C34: 0.1µF, Capacitor_SMD:C_0402_1005Metric, F.Cu at (-26.6, 30.3)
- added C35: 1µF, Capacitor_SMD:C_0603_1608Metric, F.Cu at (-20.3, 26.7)
- added C36: 4.7μF, Capacitor_SMD:C_0603_1608Metric, F.Cu at (-20.3, 29.2)
- added C37: 0.1μF, Capacitor_SMD:C_0402_1005Metric, F.Cu at (-15.5, 48.4)
- added C38: 0.1μF, Capacitor_SMD:C_0402_1005Metric, F.Cu at (-15.5, 50.4)
- added C39: 10μF, Capacitor_SMD:C_0805_2012Metric, F.Cu at (-31.6, 4.50)
- added C4: 22µF, Capacitor_SMD:C_0805_2012Metric, F.Cu at (-51.4, 34.0)
- added C40: 10μF, Capacitor_SMD:C_0805_2012Metric, F.Cu at (-31.6, 7.50)
- added C41: 0.1μF, Capacitor_SMD:C_0402_1005Metric, F.Cu at (-15.5, 52.3)
- added C42: 0.1μF, Capacitor_SMD:C_0402_1005Metric, F.Cu at (-15.5, 54.3)
- added C43: 10μF, Capacitor_SMD:C_0805_2012Metric, F.Cu at (-31.6, 10.5)
- added C44: 22μF, Capacitor_SMD:C_0603_1608Metric, F.Cu at (-12.1, 48.7)
- added C45: 22μF, Capacitor_SMD:C_0603_1608Metric, F.Cu at (-12.1, 51.2)
- added C46: 10μF, Capacitor_SMD:C_0805_2012Metric, F.Cu at (-31.6, 13.5)
- added C47: 10μF, Capacitor_SMD:C_0805_2012Metric, F.Cu at (-31.6, 16.5)
- added C48: 10μF, Capacitor_SMD:C_0805_2012Metric, F.Cu at (-31.6, 19.5)
- added C5: 0.1µF, Capacitor_SMD:C_0402_1005Metric, F.Cu at (-47.6, 15.7)
- added C51: 1µF, Capacitor_SMD:C_0603_1608Metric, F.Cu at (-54.1, 54.0)
- added C52: 1µF, Capacitor_SMD:C_0603_1608Metric, F.Cu at (-54.1, 56.5)
- added C53: 0.1μF, Capacitor_SMD:C_0402_1005Metric, F.Cu at (-66.2, 39.8)
- added C54: 0.1μF, Capacitor_SMD:C_0402_1005Metric, F.Cu at (-66.2, 41.7)
- added C55: 0.1μF, Capacitor_SMD:C_0603_1608Metric_Pad1.08x0.95mm_HandSolder, B.Cu at (88.1, 56.9)
- added C56: 0.1μF, Capacitor_SMD:C_0603_1608Metric_Pad1.08x0.95mm_HandSolder, B.Cu at (86.5, 56.9)
- added C57: 0.1μF, Capacitor_SMD:C_0603_1608Metric_Pad1.08x0.95mm_HandSolder, B.Cu at (86.5, 60.3)
- added C58: 0.1μF, Capacitor_SMD:C_0603_1608Metric_Pad1.08x0.95mm_HandSolder, B.Cu at (84.9, 57.0)
- added C59: 0.1μF, Capacitor_SMD:C_0402_1005Metric, F.Cu at (-66.2, 51.6)
- added C6: 1000pF, Capacitor_SMD:C_0402_1005Metric, F.Cu at (-47.6, 17.6)
- added C60: 0.1μF, Capacitor_SMD:C_0402_1005Metric, F.Cu at (-66.2, 53.5)
- added C61: 0.1μF, Capacitor_SMD:C_0603_1608Metric_Pad1.08x0.95mm_HandSolder, B.Cu at (69.1, 56.9)
- added C62: 0.1μF, Capacitor_SMD:C_0603_1608Metric_Pad1.08x0.95mm_HandSolder, B.Cu at (67.5, 56.9)
- added C63: 0.1μF, Capacitor_SMD:C_0603_1608Metric_Pad1.08x0.95mm_HandSolder, B.Cu at (67.5, 60.3)
- added C64: 0.1μF, Capacitor_SMD:C_0603_1608Metric_Pad1.08x0.95mm_HandSolder, B.Cu at (65.9, 56.9)
- added C65: 0.1µF, Capacitor_SMD:C_0402_1005Metric, F.Cu at (-26.6, 32.3)
- added C66: 0.1µF, Capacitor_SMD:C_0402_1005Metric, F.Cu at (-26.6, 34.3)
- added C67: 0.1µF, Capacitor_SMD:C_0402_1005Metric, F.Cu at (-26.6, 36.3)
- added C68: 0.1µF, Capacitor_SMD:C_0402_1005Metric, F.Cu at (-26.6, 38.2)
- added C69: 0.1µF, Capacitor_SMD:C_0402_1005Metric, F.Cu at (-23.8, 26.4)
- added C7: 0.1µF, Capacitor_SMD:C_0402_1005Metric, F.Cu at (-47.6, 19.6)
- added C70: 0.1µF, Capacitor_SMD:C_0402_1005Metric, F.Cu at (-23.8, 28.4)
- added C71: 0.1µF, Capacitor_SMD:C_0402_1005Metric, F.Cu at (-23.8, 30.3)
- added C72: 0.1µF, Capacitor_SMD:C_0402_1005Metric, F.Cu at (-23.8, 32.3)
- added C73: 0.1µF, Capacitor_SMD:C_0402_1005Metric, F.Cu at (106.5, 71.0)
- added C74: 0.1µF, Capacitor_SMD:C_0402_1005Metric, F.Cu at (106.5, 70.0)
- added C75: 220nF, Capacitor_SMD:C_0402_1005Metric, F.Cu at (84.0, 49.2)
- added C76: 220nF, Capacitor_SMD:C_0402_1005Metric, F.Cu at (83.0, 49.2)
- added C77: 220nF, Capacitor_SMD:C_0402_1005Metric, F.Cu at (86.0, 49.2)
- added C78: 220nF, Capacitor_SMD:C_0402_1005Metric, F.Cu at (85.0, 49.3)
- added C79: 220nF, Capacitor_SMD:C_0402_1005Metric, F.Cu at (88.0, 49.3)
- added C8: 100pF, Capacitor_SMD:C_0402_1005Metric, F.Cu at (-47.6, 21.6)
- added C80: 220nF, Capacitor_SMD:C_0402_1005Metric, F.Cu at (87.0, 49.3)
- added C81: 220nF, Capacitor_SMD:C_0402_1005Metric, F.Cu at (90.0, 49.3)
- added C82: 220nF, Capacitor_SMD:C_0402_1005Metric, F.Cu at (89.0, 49.3)
- added C83: 220nF, Capacitor_SMD:C_0402_1005Metric, F.Cu at (71.0, 49.5)
- added C84: 220nF, Capacitor_SMD:C_0402_1005Metric, F.Cu at (70.0, 49.5)
- added C85: 220nF, Capacitor_SMD:C_0402_1005Metric, F.Cu at (67.0, 49.5)
- added C86: 220nF, Capacitor_SMD:C_0402_1005Metric, F.Cu at (66.0, 49.5)
- added C87: 220nF, Capacitor_SMD:C_0402_1005Metric, F.Cu at (69.0, 49.5)
- added C88: 220nF, Capacitor_SMD:C_0402_1005Metric, F.Cu at (68.0, 49.5)
- added C89: 220nF, Capacitor_SMD:C_0402_1005Metric, F.Cu at (65.0, 49.5)
- added C9: 1000pF, Capacitor_SMD:C_0402_1005Metric, F.Cu at (-47.6, 23.6)
- added C90: 220nF, Capacitor_SMD:C_0402_1005Metric, F.Cu at (64.0, 49.5)
- added C91: 22pF, Capacitor_SMD:C_0603_1608Metric, F.Cu at (-20.3, 31.7)
- added C92: 22pF, Capacitor_SMD:C_0603_1608Metric, F.Cu at (-20.3, 34.2)
- added D1: PMEG4050EP, Diode_SMD:D_SOD-128, F.Cu at (-39.5, 21.4)
- added D2: H5VU25U, AZ1045-04F:AZ1045-04F, F.Cu at (9.00, 7.00)
- added D3: H5VU25U, AZ1045-04F:AZ1045-04F, F.Cu at (8.93, 10.5)
- added D4: H5VU25U, AZ1045-04F:AZ1045-04F, F.Cu at (9.00, 14.0)
- added D5: H5VU25U, AZ1045-04F:AZ1045-04F, F.Cu at (9.07, 22.5)
- added D6: H5VU25U, AZ1045-04F:AZ1045-04F, F.Cu at (9.00, 26.0)
- added D7: H5VU25U, AZ1045-04F:AZ1045-04F, F.Cu at (9.00, 29.5)
- added J1: 5-1775443-8, 5-1775443-8:5-1775443-8, F.Cu at (55.0, 64.0)
- added J11: Conn_02x03_Odd_Even, Connector_PinHeader_2.54mm:PinHeader_2x03_P2.54mm_Vertical, F.Cu at (-27.0, 5.32)
- added J12: USB_C_Receptacle_PowerOnly_6P, USB-C-SMD_TYPE-C-24P-QT:USB-C-SMD_TYPE-C-24P-QT, F.Cu at (-13.8, 93.9)
- added J13: Conn_02x03_Odd_Even, Connector_PinHeader_2.54mm:PinHeader_2x03_P2.54mm_Vertical, F.Cu at (-19.8, 5.32)
- added J15: Conn_01x02, Connector_PinHeader_2.54mm:PinHeader_1x02_P2.54mm_Vertical, F.Cu at (-17.5, 15.0)
- added J5: USB_C_Receptacle, USB-C-SMD_TYPE-C-24P-QT:USB-C-SMD_TYPE-C-24P-QT, F.Cu at (1.65, 10.5)
- added J6: USB_C_Receptacle, USB-C-SMD_TYPE-C-24P-QT:USB-C-SMD_TYPE-C-24P-QT, F.Cu at (1.65, 25.8)
- added J9: Conn_01x05, Connector_PinHeader_2.54mm:PinHeader_1x05_P2.54mm_Vertical, F.Cu at (-51.3, 17.0)
- added L1: 10µH, Inductor_SMD:L_Abracon_ASPI-0630LR, F.Cu at (-62.6, 18.8)
- added Q1: AOSP21321, AOSP21321:AOSP21321, F.Cu at (-44.1, 29.7)
- added Q2: BSH105,215, Package_TO_SOT_SMD:SOT-23, F.Cu at (-65.2, 25.3)
- added Q3: BSH105,215, Package_TO_SOT_SMD:SOT-23, F.Cu at (-65.2, 29.9)
- added Q4: BSH105,215, Package_TO_SOT_SMD:SOT-23, F.Cu at (-65.2, 34.5)
- added R1: 1M, Resistor_SMD:R_0805_2012Metric, F.Cu at (-41.0, 24.9)
- added R10: 9.53k, Resistor_SMD:R_0805_2012Metric_Pad1.20x1.40mm_HandSolder, F.Cu at (-60.3, 24.4)
- added R11: 100k, Resistor_SMD:R_0603_1608Metric, F.Cu at (-55.6, 28.5)
- added R12: 100k, Resistor_SMD:R_0603_1608Metric, F.Cu at (-55.6, 31.0)
- added R13: 100k, Resistor_SMD:R_0603_1608Metric, F.Cu at (-55.6, 33.5)
- added R14: 8.87k, Resistor_SMD:R_0805_2012Metric_Pad1.20x1.40mm_HandSolder, F.Cu at (-60.3, 27.3)
- added R15: 3.65k, Resistor_SMD:R_0805_2012Metric_Pad1.20x1.40mm_HandSolder, F.Cu at (-60.3, 30.3)
- added R16: 2.20k, Resistor_SMD:R_0805_2012Metric_Pad1.20x1.40mm_HandSolder, F.Cu at (-60.3, 33.2)
- added R17: 4.7k, Resistor_SMD:R_0402_1005Metric, F.Cu at (-20.9, 42.4)
- added R18: 4.7k, Resistor_SMD:R_0402_1005Metric, F.Cu at (-20.9, 44.4)
- added R19: 4.7k, Resistor_SMD:R_0402_1005Metric, F.Cu at (-18.0, 36.5)
- added R2: 10k, Resistor_SMD:R_0402_1005Metric, F.Cu at (-20.9, 36.5)
- added R20: 4.7k, Resistor_SMD:R_0402_1005Metric, F.Cu at (-18.0, 38.4)
- added R21: 12.4k, Resistor_SMD:R_0805_2012Metric_Pad1.20x1.40mm_HandSolder, F.Cu at (-26.2, 40.7)
- added R22: 10k, Resistor_SMD:R_0402_1005Metric, F.Cu at (-18.0, 40.4)
- added R23: 10k, Resistor_SMD:R_0402_1005Metric, F.Cu at (-18.0, 42.4)
- added R24: 100k, Resistor_SMD:R_0402_1005Metric, F.Cu at (-18.0, 44.4)
- added R25: 100k, Resistor_SMD:R_0402_1005Metric, F.Cu at (-15.1, 36.5)
- added R26: 100k, Resistor_SMD:R_0402_1005Metric, F.Cu at (-15.1, 38.4)
- added R27: 100k, Resistor_SMD:R_0402_1005Metric, F.Cu at (-15.1, 40.4)
- added R28: 5.1k, Resistor_SMD:R_0402_1005Metric, F.Cu at (-27.9, 20.4)
- added R29: 5.1k, Resistor_SMD:R_0402_1005Metric, F.Cu at (-27.9, 22.4)
- added R3: 47k, Resistor_SMD:R_0402_1005Metric, F.Cu at (-46.8, 3.98)
- added R30: 1k, Resistor_SMD:R_0402_1005Metric, F.Cu at (-46.8, 5.97)
- added R31: 1k, Resistor_SMD:R_0402_1005Metric, F.Cu at (-46.8, 7.96)
- added R32: 4.7k, Resistor_SMD:R_0402_1005Metric, F.Cu at (-54.7, 39.8)
- added R33: 4.7k, Resistor_SMD:R_0402_1005Metric, F.Cu at (-54.7, 41.8)
- added R34: 4.7k, Resistor_SMD:R_0402_1005Metric, F.Cu at (-54.7, 43.7)
- added R35: 1k, Resistor_SMD:R_0402_1005Metric, F.Cu at (-54.7, 45.7)
- added R36: 4.7k, Resistor_SMD:R_0402_1005Metric, F.Cu at (-46.8, 9.96)
- added R37: 4.7k, Resistor_SMD:R_0402_1005Metric, F.Cu at (-46.8, 11.9)
- added R38: 56k, Resistor_SMD:R_0402_1005Metric, F.Cu at (-54.7, 47.7)
- added R39: 4.7k, Resistor_SMD:R_0402_1005Metric, F.Cu at (-43.9, 3.98)
- added R4: 30k, Resistor_SMD:R_0603_1608Metric, F.Cu at (-55.6, 18.5)
- added R40: 4.7k, Resistor_SMD:R_0402_1005Metric, F.Cu at (-43.9, 5.97)
- added R41: 4.7k, Resistor_SMD:R_0402_1005Metric, F.Cu at (-43.9, 7.96)
- added R42: 4.7k, Resistor_SMD:R_0402_1005Metric, F.Cu at (-43.9, 9.96)
- added R43: 56k, Resistor_SMD:R_0402_1005Metric, F.Cu at (-54.7, 49.7)
- added R44: 56k, Resistor_SMD:R_0402_1005Metric, F.Cu at (-54.7, 51.7)
- added R45: 4.7k, Resistor_SMD:R_0402_1005Metric, F.Cu at (-43.9, 11.9)
- added R46: 4.7k, Resistor_SMD:R_0402_1005Metric, F.Cu at (-41.0, 3.98)
- added R47: 10k, Resistor_SMD:R_0402_1005Metric, F.Cu at (-41.0, 5.97)
- added R48: 56k, Resistor_SMD:R_0402_1005Metric, F.Cu at (-51.8, 39.8)
- added R49: 56k, Resistor_SMD:R_0402_1005Metric, F.Cu at (-51.8, 41.8)
- added R5: 100k, Resistor_SMD:R_0603_1608Metric, F.Cu at (-55.6, 21.0)
- added R50: 4.7k, Resistor_SMD:R_0402_1005Metric, F.Cu at (-51.8, 43.7)
- added R51: 1k, Resistor_SMD:R_0402_1005Metric, F.Cu at (-51.8, 45.7)
- added R52: 100k, Resistor_SMD:R_0402_1005Metric, F.Cu at (-41.0, 7.96)
- added R53: 56k, Resistor_SMD:R_0402_1005Metric, F.Cu at (-51.8, 47.7)
- added R54: 56k, Resistor_SMD:R_0402_1005Metric, F.Cu at (-51.8, 49.7)
- added R55: 56k, Resistor_SMD:R_0402_1005Metric, F.Cu at (-51.8, 51.7)
- added R56: 56k, Resistor_SMD:R_0402_1005Metric, F.Cu at (-48.9, 39.8)
- added R57: 56k, Resistor_SMD:R_0402_1005Metric, F.Cu at (-48.9, 41.8)
- added R58: 4.7k, Resistor_SMD:R_0402_1005Metric, F.Cu at (-48.9, 43.7)
- added R59: 4.7k, Resistor_SMD:R_0402_1005Metric, F.Cu at (-48.9, 45.7)
- added R6: 270, Resistor_SMD:R_0603_1608Metric, F.Cu at (-55.6, 23.5)
- added R60: 10k, Resistor_SMD:R_0402_1005Metric, F.Cu at (-22.2, 48.4)
- added R61: 0, Resistor_SMD:R_0805_2012Metric_Pad1.20x1.40mm_HandSolder, F.Cu at (-21.3, 54.9)
- added R62: 10k, Resistor_SMD:R_0402_1005Metric, F.Cu at (-22.2, 50.4)
- added R63: 10k, Resistor_SMD:R_0402_1005Metric, F.Cu at (-22.2, 52.4)
- added R64: 0, Resistor_SMD:R_0805_2012Metric_Pad1.20x1.40mm_HandSolder, F.Cu at (-21.3, 57.8)
- added R65: 3k, Resistor_SMD:R_0603_1608Metric, F.Cu at (-54.1, 59.0)
- added R66: 3k, Resistor_SMD:R_0603_1608Metric, F.Cu at (-54.1, 61.5)
- added R67: 3k, Resistor_SMD:R_0603_1608Metric, F.Cu at (-50.1, 54.0)
- added R68: 3k, Resistor_SMD:R_0603_1608Metric, F.Cu at (-50.1, 56.5)
- added R69: 3k, Resistor_SMD:R_0603_1608Metric, F.Cu at (-50.1, 59.0)
- added R7: 10k, Resistor_SMD:R_0402_1005Metric, F.Cu at (-20.9, 38.4)
- added R70: 3k, Resistor_SMD:R_0603_1608Metric, F.Cu at (-50.1, 61.5)
- added R71: 3k, Resistor_SMD:R_0603_1608Metric, F.Cu at (-46.1, 54.0)
- added R72: 3k, Resistor_SMD:R_0603_1608Metric, F.Cu at (-46.1, 56.5)
- added R73: 3k, Resistor_SMD:R_0603_1608Metric, F.Cu at (-46.1, 59.0)
- added R74: 3k, Resistor_SMD:R_0603_1608Metric, F.Cu at (-46.1, 61.5)
- added R8: 10k, Resistor_SMD:R_0402_1005Metric, F.Cu at (-20.9, 40.4)
- added R9: 11.0k, Resistor_SMD:R_0603_1608Metric, F.Cu at (-55.6, 26.0)
- added SW1: SW_Push, Button_Switch_SMD:SW_SPST_SKQG_WithStem, F.Cu at (-24.6, 16.1)
- added U1: LM3489QMM/NOPB, LM3489QMM-NOPB:LM3489QMM-NOPB, F.Cu at (-39.5, 17.0)
- added U10: SN75LVPE4410RNQR, SN75LVPE4410RNQR:SN75LVPE4410RNQR, F.Cu at (67.5, 55.0)
- added U2: TPS65987DDHRSHR, TPS65987DDHRSHR:TPS65987DDHRSHR, F.Cu at (-53.0, 7.71)
- added U4: VL822-QFN76, VL822-QFN76:VL822-QFN76, F.Cu at (130.0, 62.0)
- added U5: AP7331-10WG-7, AP7331-10WG-7:AP7331-10WG-7, F.Cu at (-33.9, 75.6)
- added U7: TPS2003CDRCR, TPS2003CDRCR:DRC10_1P65X2P40_TEX, F.Cu at (-32.1, 51.7)
- added U9: SN75LVPE4410RNQR, SN75LVPE4410RNQR:SN75LVPE4410RNQR, F.Cu at (86.5, 55.0)
- added Y1: 25MHz, Crystal:Crystal_SMD_3225-4Pin_3.2x2.5mm, F.Cu at (-31.2, 41.4)
- J10: renamed from REF**; value BUS_PCIexpress_x1 -> Bus_PCI_Express_x1
- J2, J3: renamed from REF**; value IPEX_20455-040E-76 -> 20455-040E-76
- J4: renamed from REF**; value SAMTEC_PCIE-164-02-F-D-TH-TR -> 3-2362375-4
- J7: renamed from REF**; value TE_5-5530843-0 -> Conn_02x10_Odd_Even
- J8: renamed from REF**; value 20P_Slot_Power -> Conn_02x10_Odd_Even
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Connections:
- J10 pad A1: (no net) -> unconnected-(J10-~{PRSNT1}-PadA1)
- J10 pad A10: (no net) -> Net-(J11-Pin_5)
- J10 pad A11: (no net) -> unconnected-(J10-~{PERST}-PadA11)
- J10 pad A12: (no net) -> GND
- J10 pad A13: (no net) -> unconnected-(J10-REFCLK+-PadA13)
- J10 pad A14: (no net) -> unconnected-(J10-REFCLK--PadA14)
- J10 pad A15: (no net) -> GND
- J10 pad A16: (no net) -> unconnected-(J10-PERp0-PadA16)
- J10 pad A17: (no net) -> unconnected-(J10-PERn0-PadA17)
- J10 pad A18: (no net) -> GND
- J10 pad A2: (no net) -> Net-(J11-Pin_1)
- J10 pad A3: (no net) -> Net-(J11-Pin_1)
- J10 pad A4: (no net) -> GND
- J10 pad A5: (no net) -> unconnected-(J10-JTAG2-PadA5)
- J10 pad A6: (no net) -> unconnected-(J10-JTAG3-PadA6)
- J10 pad A7: (no net) -> unconnected-(J10-JTAG4-PadA7)
- J10 pad A8: (no net) -> unconnected-(J10-JTAG5-PadA8)
- J10 pad A9: (no net) -> Net-(J11-Pin_5)
- J10 pad B1: (no net) -> Net-(J11-Pin_1)
- J10 pad B10: (no net) -> unconnected-(J10-3.3Vaux-PadB10)
- J10 pad B11: (no net) -> unconnected-(J10-~{WAKE}-PadB11)
- J10 pad B12: (no net) -> unconnected-(J10-RSVD-PadB12)
- J10 pad B13: (no net) -> GND
- J10 pad B14: (no net) -> unconnected-(J10-PETp0-PadB14)
- J10 pad B15: (no net) -> unconnected-(J10-PETn0-PadB15)
- J10 pad B16: (no net) -> GND
- J10 pad B17: (no net) -> unconnected-(J10-~{PRSNT2}-PadB17)
- J10 pad B18: (no net) -> GND
- J10 pad B2: (no net) -> Net-(J11-Pin_1)
- J10 pad B3: (no net) -> Net-(J11-Pin_1)
- J10 pad B4: (no net) -> GND
- J10 pad B5: (no net) -> unconnected-(J10-SMCLK-PadB5)
- J10 pad B6: (no net) -> unconnected-(J10-SMDAT-PadB6)
- J10 pad B7: (no net) -> GND
- J10 pad B8: (no net) -> Net-(J11-Pin_5)
- J10 pad B9: (no net) -> unconnected-(J10-JTAG1-PadB9)
- J2 pad 1: (no net) -> /RX6N
- J2 pad 10: (no net) -> /TX4N
- J2 pad 11: (no net) -> /TX4P
- J2 pad 12: (no net) -> GND
- J2 pad 13: (no net) -> /RX4N
- J2 pad 14: (no net) -> /RX4P
- J2 pad 15: (no net) -> GND
- J2 pad 16: (no net) -> /TX3N
- J2 pad 17: (no net) -> /TX3P
- J2 pad 18: (no net) -> GND
- J2 pad 19: (no net) -> /RX3N
- J2 pad 2: (no net) -> /RX6P
- J2 pad 20: (no net) -> /RX3P
- J2 pad 21: (no net) -> GND
- J2 pad 22: (no net) -> /TX2N
- J2 pad 23: (no net) -> /TX2P
- J2 pad 24: (no net) -> GND
- J2 pad 25: (no net) -> /RX2N
- J2 pad 26: (no net) -> /RX2P
- J2 pad 27: (no net) -> GND
- J2 pad 28: (no net) -> /TX1N
- J2 pad 29: (no net) -> /TX1P
- J2 pad 3: (no net) -> GND
- J2 pad 30: (no net) -> GND
- J2 pad 31: (no net) -> /RX1N
- J2 pad 32: (no net) -> /RX1P
- J2 pad 33: (no net) -> GND
- J2 pad 34: (no net) -> /TX0N
- J2 pad 35: (no net) -> /TX0P
- J2 pad 36: (no net) -> GND
- J2 pad 37: (no net) -> /RX0N
- J2 pad 38: (no net) -> /RX0P
- J2 pad 39: (no net) -> GND
- J2 pad 4: (no net) -> /TX5N
- J2 pad 40: (no net) -> /DET2
- J2 pad 5: (no net) -> /TX5P
- J2 pad 6: (no net) -> GND
- J2 pad 7: (no net) -> /RX5N
- J2 pad 8: (no net) -> /RX5P
- J2 pad 9: (no net) -> GND
- J2 pad S1: (no net) -> GND
- J2 pad S2: (no net) -> GND
- J2 pad S3: (no net) -> GND
- J2 pad S4: (no net) -> GND
- J3 pad 1: (no net) -> unconnected-(J3-Pad1)
- J3 pad 10: (no net) -> Net-(J3-Pad10)
- J3 pad 11: (no net) -> Net-(J3-CON_DET)
- J3 pad 12: (no net) -> /PWREN
- J3 pad 13: (no net) -> /RST
- J3 pad 14: (no net) -> /PWROK
- J3 pad 15: (no net) -> Net-(J3-P_AC_LOSS)
- J3 pad 16: (no net) -> Net-(J3-MCU_IRQ#)
- J3 pad 17: (no net) -> GND
- J3 pad 18: (no net) -> /SMDAT
- J3 pad 19: (no net) -> /SMCLK
- J3 pad 2: (no net) -> unconnected-(J3-Pad2)
- J3 pad 20: (no net) -> GND
- J3 pad 21: (no net) -> /C_DN
- J3 pad 22: (no net) -> /C_DP
- J3 pad 23: (no net) -> GND
- J3 pad 24: (no net) -> /C_TXN
- J3 pad 25: (no net) -> /C_TXP
- J3 pad 26: (no net) -> GND
- J3 pad 27: (no net) -> /C_RXN
- J3 pad 28: (no net) -> /C_RXP
- J3 pad 29: (no net) -> GND
- J3 pad 3: (no net) -> unconnected-(J3-Pad3)
- J3 pad 30: (no net) -> /CLKN
- J3 pad 31: (no net) -> /CLKP
- J3 pad 32: (no net) -> GND
- J3 pad 33: (no net) -> /TX7N
- J3 pad 34: (no net) -> /TX7P
- J3 pad 35: (no net) -> GND
- J3 pad 36: (no net) -> /RX7N
- J3 pad 37: (no net) -> /RX7P
- J3 pad 38: (no net) -> GND
- J3 pad 39: (no net) -> /TX6N
- J3 pad 4: (no net) -> unconnected-(J3-Pad4)
- J3 pad 40: (no net) -> /TX6P
- J3 pad 5: (no net) -> unconnected-(J3-Pad5)
- J3 pad 6: (no net) -> unconnected-(J3-Pad6)
- J3 pad 7: (no net) -> unconnected-(J3-Pad7)
- J3 pad 8: (no net) -> unconnected-(J3-Pad8)
- J3 pad 9: (no net) -> /DET1
- J3 pad S1: (no net) -> GND
- J3 pad S2: (no net) -> GND
- J3 pad S3: (no net) -> GND
- J3 pad S4: (no net) -> GND
- J4 pad A1: (no net) -> unconnected-(J4-PadA1)
- J4 pad A10: (no net) -> +3V3
- J4 pad A11: (no net) -> /PERST
- J4 pad A12: (no net) -> GND
- J4 pad A13: (no net) -> /CLKP
- J4 pad A14: (no net) -> /CLKN
- J4 pad A15: (no net) -> GND
- J4 pad A16: (no net) -> /RX0P
- J4 pad A17: (no net) -> /RX0N
- J4 pad A18: (no net) -> GND
- J4 pad A19: (no net) -> unconnected-(J4-PadA19)
- J4 pad A2: (no net) -> /+12V0
- J4 pad A20: (no net) -> GND
- J4 pad A21: (no net) -> /RX1P
- J4 pad A22: (no net) -> /RX1N
- J4 pad A23: (no net) -> GND
- J4 pad A24: (no net) -> GND
- J4 pad A25: (no net) -> /RX2P
- J4 pad A26: (no net) -> /RX2N
- J4 pad A27: (no net) -> GND
- J4 pad A28: (no net) -> GND
- J4 pad A29: (no net) -> /RX3P
- J4 pad A3: (no net) -> /+12V0
- J4 pad A30: (no net) -> /RX3N
- J4 pad A31: (no net) -> GND
- J4 pad A32: (no net) -> unconnected-(J4-PadA32)
- J4 pad A33: (no net) -> unconnected-(J4-PadA33)
- J4 pad A34: (no net) -> GND
- J4 pad A35: (no net) -> /RX4P
- J4 pad A36: (no net) -> /RX4N
- J4 pad A37: (no net) -> GND
- J4 pad A38: (no net) -> GND
- J4 pad A39: (no net) -> /RX5P
- J4 pad A4: (no net) -> GND
- J4 pad A40: (no net) -> /RX5N
- J4 pad A41: (no net) -> GND
- J4 pad A42: (no net) -> GND
- J4 pad A43: (no net) -> /RX6P
- J4 pad A44: (no net) -> /RX6N
- J4 pad A45: (no net) -> GND
- J4 pad A46: (no net) -> GND
- J4 pad A47: (no net) -> /RX7P
- J4 pad A48: (no net) -> /RX7N
- J4 pad A49: (no net) -> GND
- J4 pad A5: (no net) -> unconnected-(J4-PadA5)
- J4 pad A50: (no net) -> unconnected-(J4-PadA50)
- J4 pad A51: (no net) -> GND
- J4 pad A52: (no net) -> unconnected-(J4-PadA52)
- J4 pad A53: (no net) -> unconnected-(J4-PadA53)
- J4 pad A54: (no net) -> GND
- J4 pad A55: (no net) -> GND
- J4 pad A56: (no net) -> unconnected-(J4-PadA56)
- J4 pad A57: (no net) -> unconnected-(J4-PadA57)
- J4 pad A58: (no net) -> GND
- J4 pad A59: (no net) -> GND
- J4 pad A6: (no net) -> unconnected-(J4-PadA6)
- J4 pad A60: (no net) -> unconnected-(J4-PadA60)
- J4 pad A61: (no net) -> unconnected-(J4-PadA61)
- J4 pad A62: (no net) -> GND
- J4 pad A63: (no net) -> GND
- J4 pad A64: (no net) -> unconnected-(J4-PadA64)
- J4 pad A65: (no net) -> unconnected-(J4-PadA65)
- J4 pad A66: (no net) -> GND
- J4 pad A67: (no net) -> GND
- J4 pad A68: (no net) -> unconnected-(J4-PadA68)
- J4 pad A69: (no net) -> unconnected-(J4-PadA69)
- J4 pad A7: (no net) -> unconnected-(J4-PadA7)
- J4 pad A70: (no net) -> GND
- J4 pad A71: (no net) -> GND
- J4 pad A72: (no net) -> unconnected-(J4-PadA72)
- J4 pad A73: (no net) -> unconnected-(J4-PadA73)
- J4 pad A74: (no net) -> GND
- J4 pad A75: (no net) -> GND
- J4 pad A76: (no net) -> unconnected-(J4-PadA76)
- J4 pad A77: (no net) -> unconnected-(J4-PadA77)
- J4 pad A78: (no net) -> GND
- J4 pad A79: (no net) -> GND
- J4 pad A8: (no net) -> unconnected-(J4-PadA8)
- J4 pad A80: (no net) -> unconnected-(J4-PadA80)
- J4 pad A81: (no net) -> unconnected-(J4-PadA81)
- J4 pad A82: (no net) -> GND
- J4 pad A9: (no net) -> +3V3
- J4 pad B1: (no net) -> /+12V0
- J4 pad B10: (no net) -> +3V3
- J4 pad B11: (no net) -> unconnected-(J4-PadB11)
- J4 pad B12: (no net) -> /CLKREQ
- J4 pad B13: (no net) -> GND
- J4 pad B14: (no net) -> /TX0RP
- J4 pad B15: (no net) -> /TX0RN
- J4 pad B16: (no net) -> GND
- J4 pad B17: (no net) -> unconnected-(J4-PadB17)
- J4 pad B18: (no net) -> GND
- J4 pad B19: (no net) -> /TX1RP
- J4 pad B2: (no net) -> /+12V0
- J4 pad B20: (no net) -> /TX1RN
- J4 pad B21: (no net) -> GND
- J4 pad B22: (no net) -> GND
- J4 pad B23: (no net) -> /TX2RP
- J4 pad B24: (no net) -> /TX2RN
- J4 pad B25: (no net) -> GND
- J4 pad B26: (no net) -> GND
- J4 pad B27: (no net) -> /TX3RP
- J4 pad B28: (no net) -> /TX3RN
- J4 pad B29: (no net) -> GND
- J4 pad B3: (no net) -> /+12V0
- J4 pad B30: (no net) -> unconnected-(J4-PadB30)
- J4 pad B31: (no net) -> unconnected-(J4-PadB31)
- J4 pad B32: (no net) -> GND
- J4 pad B33: (no net) -> /TX4RP
- J4 pad B34: (no net) -> /TX4RN
- J4 pad B35: (no net) -> GND
- J4 pad B36: (no net) -> GND
- J4 pad B37: (no net) -> /TX5RP
- J4 pad B38: (no net) -> /TX5RN
- J4 pad B39: (no net) -> GND
- J4 pad B4: (no net) -> GND
- J4 pad B40: (no net) -> GND
- J4 pad B41: (no net) -> /TX6RP
- J4 pad B42: (no net) -> /TX6RN
- J4 pad B43: (no net) -> GND
- J4 pad B44: (no net) -> GND
- J4 pad B45: (no net) -> /TX7RP
- J4 pad B46: (no net) -> /TX7RN
- J4 pad B47: (no net) -> GND
- J4 pad B48: (no net) -> unconnected-(J4-PadB48)
- J4 pad B49: (no net) -> GND
- J4 pad B5: (no net) -> /SMCLK
- J4 pad B50: (no net) -> unconnected-(J4-PadB50)
- J4 pad B51: (no net) -> unconnected-(J4-PadB51)
- J4 pad B52: (no net) -> GND
- J4 pad B53: (no net) -> GND
- J4 pad B54: (no net) -> unconnected-(J4-PadB54)
- J4 pad B55: (no net) -> unconnected-(J4-PadB55)
- J4 pad B56: (no net) -> GND
- J4 pad B57: (no net) -> GND
- J4 pad B58: (no net) -> unconnected-(J4-PadB58)
- J4 pad B59: (no net) -> unconnected-(J4-PadB59)
- J4 pad B6: (no net) -> /SMDAT
- J4 pad B60: (no net) -> GND
- J4 pad B61: (no net) -> GND
- J4 pad B62: (no net) -> unconnected-(J4-PadB62)
- J4 pad B63: (no net) -> unconnected-(J4-PadB63)
- J4 pad B64: (no net) -> GND
- J4 pad B65: (no net) -> GND
- J4 pad B66: (no net) -> unconnected-(J4-PadB66)
- J4 pad B67: (no net) -> unconnected-(J4-PadB67)
- J4 pad B68: (no net) -> GND
- J4 pad B69: (no net) -> GND
- J4 pad B7: (no net) -> GND
- J4 pad B70: (no net) -> unconnected-(J4-PadB70)
- J4 pad B71: (no net) -> unconnected-(J4-PadB71)
- J4 pad B72: (no net) -> GND
- J4 pad B73: (no net) -> GND
- J4 pad B74: (no net) -> unconnected-(J4-PadB74)
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Routing:
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- removed copper zone on B.Cu, net (none)
- removed copper zone on F.Cu, net (none)
Other:
- copper layers 2 -> 4
- board text added: "${REFERENCE}"

Commit message: Continue working on board layout
Parts:
- added R75: 4.7k, Resistor_SMD:R_0402_1005Metric, F.Cu at (119.0, 55.5)
- added R76: 10k, Resistor_SMD:R_0402_1005Metric, F.Cu at (119.0, 54.5)
- added R77: 2M, Resistor_SMD:R_0603_1608Metric, F.Cu at (121.0, 55.5)
- moved C10 178.6 mm to (142.2, 64.0)
- moved C11 177.9 mm to (142.2, 62.8)
- moved U5 177.4 mm to (142.0, 52.0), turned to 180 degrees
- moved C12 177.3 mm to (142.2, 61.6)
- moved C13 176.8 mm to (142.2, 60.4)
- moved C14 176.3 mm to (142.2, 59.2)
- moved C28 170.9 mm to (137.4, 69.2), turned to -90 degrees
- moved C15 170.4 mm to (137.0, 54.8), turned to 90 degrees
- moved C16 169.0 mm to (135.8, 54.8), turned to 90 degrees
- moved C29 168.2 mm to (135.0, 69.2), turned to -90 degrees
- moved C17 166.5 mm to (134.6, 54.8), turned to 90 degrees
- moved R8 165.1 mm to (142.2, 66.0)
- moved C19 165.0 mm to (133.4, 54.8), turned to 90 degrees
- moved C30 164.8 mm to (132.0, 69.2), turned to -90 degrees
- moved C36 164.4 mm to (142.0, 55.0), turned to 180 degrees
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Connections:
- C67 pad 1: /USB C DFPs/USB_DFP0_TX2P -> /USB C DFPs/USB_DFP0_TX2N
- C68 pad 1: /USB C DFPs/USB_DFP0_TX2N -> /USB C DFPs/USB_DFP0_TX2P
- C71 pad 1: /USB C DFPs/USB_DFP1_TX2P -> /USB C DFPs/USB_DFP1_TX2N
- C72 pad 1: /USB C DFPs/USB_DFP1_TX2N -> /USB C DFPs/USB_DFP1_TX2P
- D2 pad 10: unconnected-(D2-NC-Pad10) -> /USB C DFPs/USB_DFP0_TX1P
- D2 pad 6: unconnected-(D2-NC-Pad6) -> /USB C DFPs/USB_DFP0_RX1N
- D2 pad 7: unconnected-(D2-NC-Pad7) -> /USB C DFPs/USB_DFP0_RX1P
- D2 pad 8: unconnected-(D2-GND-Pad8) -> GND
- D2 pad 9: unconnected-(D2-NC-Pad9) -> /USB C DFPs/USB_DFP0_TX1N
- D3 pad 10: unconnected-(D3-NC-Pad10) -> /USB C DFPs/USB_DFP0_D1P
- D3 pad 6: unconnected-(D3-NC-Pad6) -> /USB C DFPs/USB_DFP0_TX2P
- D3 pad 7: unconnected-(D3-NC-Pad7) -> /USB C DFPs/USB_DFP0_TX2N
- D3 pad 8: unconnected-(D3-GND-Pad8) -> GND
- D3 pad 9: unconnected-(D3-NC-Pad9) -> /USB C DFPs/USB_DFP0_D1N
- D4 pad 10: unconnected-(D4-NC-Pad10) -> /USB C DFPs/USB_DFP0_RX2N
- D4 pad 6: unconnected-(D4-NC-Pad6) -> /USB C DFPs/USB_DFP0_D2N
- D4 pad 7: unconnected-(D4-NC-Pad7) -> /USB C DFPs/USB_DFP0_D2P
- D4 pad 8: unconnected-(D4-GND-Pad8) -> GND
- D4 pad 9: unconnected-(D4-NC-Pad9) -> /USB C DFPs/USB_DFP0_RX2P
- D5 pad 10: unconnected-(D5-NC-Pad10) -> /USB C DFPs/USB_DFP1_D2P
- D5 pad 6: unconnected-(D5-NC-Pad6) -> /USB C DFPs/USB_DFP1_TX1N
- D5 pad 7: unconnected-(D5-NC-Pad7) -> /USB C DFPs/USB_DFP1_TX1P
- D5 pad 8: unconnected-(D5-GND-Pad8) -> GND
- D5 pad 9: unconnected-(D5-NC-Pad9) -> /USB C DFPs/USB_DFP1_D2N
- D6 pad 10: unconnected-(D6-NC-Pad10) -> /USB C DFPs/USB_DFP1_RX1P
- D6 pad 6: unconnected-(D6-NC-Pad6) -> /USB C DFPs/USB_DFP1_TX2P
- D6 pad 7: unconnected-(D6-NC-Pad7) -> /USB C DFPs/USB_DFP1_TX2N
- D6 pad 8: unconnected-(D6-GND-Pad8) -> GND
- D6 pad 9: unconnected-(D6-NC-Pad9) -> /USB C DFPs/USB_DFP1_RX1N
- D7 pad 10: unconnected-(D7-NC-Pad10) -> /USB C DFPs/USB_DFP1_RX2N
- D7 pad 6: unconnected-(D7-NC-Pad6) -> /USB C DFPs/USB_DFP1_D1N
- D7 pad 7: unconnected-(D7-NC-Pad7) -> /USB C DFPs/USB_DFP1_D1P
- D7 pad 8: unconnected-(D7-GND-Pad8) -> GND
- D7 pad 9: unconnected-(D7-NC-Pad9) -> /USB C DFPs/USB_DFP1_RX2P
- U4 pad 10: /USB Hub/USB_DFP0_DN -> /USB C DFPs/USB_DFP0_D1N
- U4 pad 15: /USB C DFPs/USB_DFP0_RX2P -> /USB C DFPs/USB_DFP0_RX2N
- U4 pad 16: /USB C DFPs/USB_DFP0_RX2N -> /USB C DFPs/USB_DFP0_RX2P
- U4 pad 18: /USB Hub/USB_DFP1_DP -> /USB C DFPs/USB_DFP0_D2P
- U4 pad 19: /USB Hub/USB_DFP1_DN -> /USB C DFPs/USB_DFP0_D2N
- U4 pad 22: /USB Hub/USB_DFP2_DP -> /USB C DFPs/USB_DFP1_D2P
- U4 pad 23: /USB Hub/USB_DFP2_DN -> /USB C DFPs/USB_DFP1_D2N
- U4 pad 34: /USB C DFPs/USB_DFP1_RX2P -> /USB C DFPs/USB_DFP1_RX2N
- U4 pad 35: /USB C DFPs/USB_DFP1_RX2N -> /USB C DFPs/USB_DFP1_RX2P
- U4 pad 37: /USB Hub/USB_DFP3_DP -> /USB C DFPs/USB_DFP1_D1P
- U4 pad 38: /USB Hub/USB_DFP3_DN -> /USB C DFPs/USB_DFP1_D1N
- U4 pad 9: /USB Hub/USB_DFP0_DP -> /USB C DFPs/USB_DFP0_D1P
- Y1 pad 2: /USB Hub/XO -> GND
- Y1 pad 3: (no net) -> /USB Hub/XO
- Y1 pad 4: (no net) -> GND
Routing:
- net /USB Hub/SSTX1+: track 0.00 -> 141.4 mm, vias 0 -> 2
- net /USB Hub/SSTX1-: track 0.00 -> 140.5 mm, vias 0 -> 2
- net /USB C DFPs/USB_DFP0_RX1P: track 9.83 -> 149.5 mm, vias 2 -> 4
- net /USB C DFPs/USB_DFP0_RX1N: track 9.84 -> 148.6 mm, vias 2 -> 4
- net /USB C DFPs/USB_DFP0_D1P: track 4.73 -> 141.0 mm, vias 0 -> 2
- net /USB C DFPs/USB_DFP0_D1N: track 4.73 -> 140.1 mm, vias 0 -> 2
- net /USB Hub/SSTX2+: track 0.00 -> 131.0 mm, vias 0 -> 2
- net /USB Hub/SSTX2-: track 0.00 -> 130.1 mm, vias 0 -> 2
- net /USB C DFPs/USB_DFP0_RX2N: track 4.68 -> 133.9 mm, vias 0 -> 2
- net /USB C DFPs/USB_DFP0_RX2P: track 4.68 -> 133.0 mm, vias 0 -> 2
- net /USB C DFPs/USB_DFP0_D2P: track 15.7 -> 141.4 mm, vias 2 -> 4
- net /USB C DFPs/USB_DFP0_D2N: track 15.8 -> 140.6 mm, vias 2 -> 4
- net /USB C DFPs/USB_DFP1_D2P: track 16.2 -> 136.8 mm, vias 2 -> 4
- net /USB C DFPs/USB_DFP1_D2N: track 16.1 -> 136.4 mm, vias 2 -> 4
- net /USB C DFPs/USB_DFP1_RX1P: track 9.37 -> 112.2 mm, vias 2 -> 4
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- added copper zone on F.Cu, net +3V3
- added copper zone on In1.Cu, net +3V3
Other:
- board size 172.2 x 76.7 mm -> 174.7 x 76.7 mm

Commit message: Lay out more components
Parts:
- removed C57, C62: 0.1μF, Capacitor_SMD:C_0603_1608Metric_Pad1.08x0.95mm_HandSolder
- added J14: ATX-24, 1-1775099-3:1-1775099-3, F.Cu at (90.8, 6.21)
- added J16: 20V 5A DC, Connector_BarrelJack:BarrelJack_CUI_PJ-063AH_Horizontal, F.Cu at (12.0, 51.5)
- added JP1: SolderJumper_2_Open, Jumper:SolderJumper-2_P1.3mm_Open_TrianglePad1.0x1.5mm, F.Cu at (142.0, 15.0)
- added JP10: SolderJumper_2_Open, Jumper:SolderJumper-2_P1.3mm_Open_TrianglePad1.0x1.5mm, F.Cu at (81.5, 15.0)
- added JP2: SolderJumper_2_Open, Jumper:SolderJumper-2_P1.3mm_Open_TrianglePad1.0x1.5mm, F.Cu at (137.5, 15.0)
- added JP3: SolderJumper_2_Open, Jumper:SolderJumper-2_P1.3mm_Open_TrianglePad1.0x1.5mm, F.Cu at (133.0, 15.0)
- added JP4: SolderJumper_2_Open, Jumper:SolderJumper-2_P1.3mm_Open_TrianglePad1.0x1.5mm, F.Cu at (128.5, 15.0)
- added JP5: SolderJumper_2_Open, Jumper:SolderJumper-2_P1.3mm_Open_TrianglePad1.0x1.5mm, F.Cu at (124.0, 15.0)
- added JP6: SolderJumper_2_Open, Jumper:SolderJumper-2_P1.3mm_Open_TrianglePad1.0x1.5mm, F.Cu at (99.5, 15.0)
- added JP7: SolderJumper_2_Open, Jumper:SolderJumper-2_P1.3mm_Open_TrianglePad1.0x1.5mm, F.Cu at (95.0, 15.0)
- added JP8: SolderJumper_2_Open, Jumper:SolderJumper-2_P1.3mm_Open_TrianglePad1.0x1.5mm, F.Cu at (90.5, 15.0)
- added JP9: SolderJumper_2_Open, Jumper:SolderJumper-2_P1.3mm_Open_TrianglePad1.0x1.5mm, F.Cu at (86.0, 15.0)
- added TP1: TestPoint_Small, TestPoint:TestPoint_Pad_D1.0mm, F.Cu at (119.0, 74.0)
- added TP10: TestPoint_Small, TestPoint:TestPoint_Pad_D1.0mm, F.Cu at (96.5, 74.0)
- added TP11: TestPoint_Small, TestPoint:TestPoint_Pad_D1.0mm, F.Cu at (89.0, 74.0)
- added TP12: TestPoint_Small, TestPoint:TestPoint_Pad_D1.0mm, F.Cu at (91.5, 74.0)
- added TP13: TestPoint_Small, TestPoint:TestPoint_Pad_D1.0mm, F.Cu at (94.0, 74.0)
- added TP2: TestPoint_Small, TestPoint:TestPoint_Pad_D1.0mm, F.Cu at (116.5, 74.0)
- added TP3: TestPoint_Small, TestPoint:TestPoint_Pad_D1.0mm, F.Cu at (114.0, 74.0)
- added TP4: TestPoint_Small, TestPoint:TestPoint_Pad_D1.0mm, F.Cu at (111.5, 74.0)
- added TP5: TestPoint_Small, TestPoint:TestPoint_Pad_D1.0mm, F.Cu at (109.0, 74.0)
- added TP6: TestPoint_Small, TestPoint:TestPoint_Pad_D1.0mm, F.Cu at (106.5, 74.0)
- added TP7: TestPoint_Small, TestPoint:TestPoint_Pad_D1.0mm, F.Cu at (104.0, 74.0)
- added TP8: TestPoint_Small, TestPoint:TestPoint_Pad_D1.0mm, F.Cu at (101.5, 74.0)
- added TP9: TestPoint_Small, TestPoint:TestPoint_Pad_D1.0mm, F.Cu at (99.0, 74.0)
- C55, C56, C58, C61, C63, C64: footprint Capacitor_SMD:C_0603_1608Metric_Pad1.08x0.95mm_HandSolder -> Capacitor_SMD:C_0402_1005Metric; moved to F.Cu
- J11: moved to B.Cu
- R38, R43, R44, R48, R49, R53, R54, R55, R56, R57: value 56k -> 47k
- R65, R66, R67, R68, R69, R70, R71, R72, R73, R74: value 3k -> 12k; footprint Resistor_SMD:R_0603_1608Metric -> Resistor_SMD:R_0402_1005Metric
- moved J11 189.0 mm to (161.4, 19.0)
- moved J12 185.6 mm to (149.9, 6.48), turned to 90 degrees
- moved C39 176.2 mm to (144.5, 10.5), turned to 180 degrees
- moved C40 176.2 mm to (144.5, 2.50), turned to 180 degrees
- moved R29 173.6 mm to (145.0, 7.00), turned to 180 degrees
- moved R28 173.5 mm to (145.0, 6.00), turned to 180 degrees
- moved C43 162.8 mm to (131.1, 2.50), turned to 180 degrees
- moved J13 159.9 mm to (140.0, 3.00), turned to -90 degrees
- moved C53 158.1 mm to (91.5, 51.5)
- moved C54 148.0 mm to (81.5, 51.5), turned to 180 degrees
- moved R65 147.7 mm to (93.5, 54.5)
- moved R33 146.8 mm to (91.5, 55.5)
- moved R34 146.7 mm to (91.5, 56.5)
- moved R35 146.6 mm to (91.5, 57.5), turned to 180 degrees
- moved R44 146.2 mm to (91.5, 54.5)
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Connections:
- net /+12V0 renamed +12V
- C40 pad 2: Net-(J13-Pin_1) -> Net-(J13-Pin_2)
- C41 pad 1: Net-(C41-Pad1) -> +5V
- C43 pad 1: Net-(J13-Pin_5) -> Net-(J13-Pin_6)
- C44 pad 1: /USB C DFPs/USB_DFP1_VBUS -> /USB C DFPs/USB_DFP0_VBUS
- C45 pad 1: /USB C DFPs/USB_DFP0_VBUS -> /USB C DFPs/USB_DFP1_VBUS
- J10 pad A10: Net-(J11-Pin_5) -> Net-(J11-Pin_6)
- J10 pad A2: Net-(J11-Pin_1) -> Net-(J11-Pin_2)
- J10 pad A3: Net-(J11-Pin_1) -> Net-(J11-Pin_2)
- J10 pad A9: Net-(J11-Pin_5) -> Net-(J11-Pin_6)
- J10 pad B1: Net-(J11-Pin_1) -> Net-(J11-Pin_2)
- J10 pad B2: Net-(J11-Pin_1) -> Net-(J11-Pin_2)
- J10 pad B3: Net-(J11-Pin_1) -> Net-(J11-Pin_2)
- J10 pad B8: Net-(J11-Pin_5) -> Net-(J11-Pin_6)
- J11 pad 1: Net-(J11-Pin_1) -> GND
- J11 pad 2: GND -> Net-(J11-Pin_2)
- J11 pad 3: Net-(J11-Pin_1) -> GND
- J11 pad 4: GND -> Net-(J11-Pin_2)
- J11 pad 5: Net-(J11-Pin_5) -> GND
- J11 pad 6: GND -> Net-(J11-Pin_6)
- J13 pad 1: Net-(J13-Pin_1) -> GND
- J13 pad 2: GND -> Net-(J13-Pin_2)
- J13 pad 3: Net-(J13-Pin_1) -> GND
- J13 pad 4: GND -> Net-(J13-Pin_2)
- J13 pad 5: Net-(J13-Pin_5) -> GND
- J13 pad 6: GND -> Net-(J13-Pin_6)
- U4 pad 77: unconnected-(U4-EP-Pad77) -> GND
- U7 pad 10: /USB Hub/USB_DFP0_FLT -> /USB Hub/USB_DFP2_FLT
- U7 pad 3: Net-(C41-Pad1) -> +5V
- U7 pad 4: /USB Hub/USB_DFP0_EN -> /USB Hub/USB_DFP2_EN
- U7 pad 5: /USB Hub/USB_DFP2_EN -> /USB Hub/USB_DFP0_EN
- U7 pad 6: /USB Hub/USB_DFP2_FLT -> /USB Hub/USB_DFP0_FLT
- U7 pad 8: /USB C DFPs/USB_DFP1_VBUS -> /USB C DFPs/USB_DFP0_VBUS
- U7 pad 9: /USB C DFPs/USB_DFP0_VBUS -> /USB C DFPs/USB_DFP1_VBUS
Routing:
- net +3V3: track 85.9 -> 531.4 mm, vias 15 -> 48
- net +5V: track 0.00 -> 207.4 mm, vias 0 -> 18
- net /USB Hub/USB_DFP0_FLT: track 5.17 -> 172.3 mm, vias 0 -> 6
- net /USB Hub/USB_DFP0_EN: track 2.45 -> 166.5 mm, vias 0 -> 6
- net /USB Hub/USB_DFP2_FLT: track 5.43 -> 164.1 mm, vias 0 -> 6
- net /USB Hub/USB_DFP2_EN: track 2.41 -> 150.6 mm, vias 0 -> 4
- net /SMCLK: track 0.00 -> 95.1 mm, vias 0 -> 2
- net /PWR_SW: track 0.00 -> 92.7 mm, vias 0 -> 2
- net /SMDAT: track 0.00 -> 90.9 mm, vias 0 -> 2
- net Net-(JP6-A): track 0.00 -> 87.5 mm
- net Net-(J11-Pin_2): track 0.00 -> 75.3 mm
- net Net-(JP10-A): track 0.00 -> 62.8 mm, vias 0 -> 1
- net /CLKREQ: track 0.00 -> 61.7 mm, vias 0 -> 1
- net /USB C DFPs/USB_DFP0_RX1N: track 148.6 -> 206.9 mm
- net /USB C DFPs/USB_DFP0_RX2P: track 133.0 -> 191.1 mm
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- added copper zone on F.Cu, net +12V
- added copper zone on In1.Cu, net +20V
- added copper zone on B.Cu, net GND
- added copper zone on F.Cu, net GND
- added copper zone on In1.Cu, net GND
- added copper zone on In2.Cu, net GND
- removed copper zone on F.Cu, net +3V3

Commit message: Updated board layout
Parts:
- removed C1, C2: 47µF, Capacitor_Tantalum_SMD:CP_EIA-7343-43_Kemet-X
- removed C18: 220pF, Capacitor_SMD:C_0201_0603Metric
- removed C20, C5, C7: 0.1µF, Capacitor_SMD:C_0402_1005Metric
- removed C21: 1µF, Capacitor_SMD:C_0603_1608Metric
- removed C22, C23, C24, C25, C26: 10µF, Capacitor_SMD:C_0402_1005Metric
- removed C3, C4: 22µF, Capacitor_SMD:C_0805_2012Metric
- removed C6, C9: 1000pF, Capacitor_SMD:C_0402_1005Metric
- removed C8: 100pF, Capacitor_SMD:C_0402_1005Metric
- removed D1: PMEG4050EP, Diode_SMD:D_SOD-128
- removed J9: Conn_01x05, Connector_PinHeader_2.54mm:PinHeader_1x05_P2.54mm_Vertical
- removed L1: 10µH, Inductor_SMD:L_Abracon_ASPI-0630LR
- removed Q1: AOSP21321, AOSP21321:AOSP21321
- removed Q2, Q3, Q4: BSH105,215, Package_TO_SOT_SMD:SOT-23
- removed R1: 1M, Resistor_SMD:R_0805_2012Metric
- removed R10: 9.53k, Resistor_SMD:R_0805_2012Metric_Pad1.20x1.40mm_HandSolder
- removed R11, R12, R13, R5: 100k, Resistor_SMD:R_0603_1608Metric
- removed R14: 8.87k, Resistor_SMD:R_0805_2012Metric_Pad1.20x1.40mm_HandSolder
- removed R15: 3.65k, Resistor_SMD:R_0805_2012Metric_Pad1.20x1.40mm_HandSolder
- removed R16: 2.20k, Resistor_SMD:R_0805_2012Metric_Pad1.20x1.40mm_HandSolder
- removed R3: 47k, Resistor_SMD:R_0402_1005Metric
- removed R30, R31: 1k, Resistor_SMD:R_0402_1005Metric
- removed R36, R37, R39, R40, R41, R42, R45, R46: 4.7k, Resistor_SMD:R_0402_1005Metric
- removed R4: 30k, Resistor_SMD:R_0603_1608Metric
- removed R47: 10k, Resistor_SMD:R_0402_1005Metric
- removed R52: 100k, Resistor_SMD:R_0402_1005Metric
- removed R6: 270, Resistor_SMD:R_0603_1608Metric
- removed R9: 11.0k, Resistor_SMD:R_0603_1608Metric
- removed U1: LM3489QMM/NOPB, LM3489QMM-NOPB:LM3489QMM-NOPB
- removed U2: TPS65987DDHRSHR, TPS65987DDHRSHR:TPS65987DDHRSHR
- added J17: 8730, KEYSTONE_8730:KEYSTONE_8730, F.Cu at (42.0, 59.0)
- J11: footprint Connector_PinHeader_2.54mm:PinHeader_2x03_P2.54mm_Vertical -> Connector_PinHeader_2.54mm:PinHeader_1x06_P2.54mm_Vertical; moved to F.Cu
- moved C37 47.6 mm to (3.00, 4.50), turned to 180 degrees
- moved C38 26.4 mm to (3.00, 31.5), turned to 180 degrees
- moved J8 16.1 mm to (39.8, 76.8)
- moved J10 8.49 mm to (167.5, 26.0)
- moved J1 6.05 mm to (56.2, 64.8)
- moved J11 4.10 mm to (160.0, 22.9), turned to 180 degrees
- moved C73 0.30 mm to (106.5, 70.7)
- moved C74 0.30 mm to (106.5, 69.7)
Connections:
- ? pad 1: (no net) -> GND (x2)
- REF** pad 1: (no net) -> GND (x4)
- U5 pad 2: unconnected-(U5-GND-Pad2) -> GND
Routing:
- net Net-(J7-Pin_20): track 0.00 -> 83.3 mm
- net Net-(J7-Pin_18): track 0.00 -> 82.6 mm
- net /PWR_SW: track 92.7 -> 171.0 mm, vias 2 -> 3
- net Net-(J7-Pin_17): track 0.00 -> 77.7 mm, vias 0 -> 1
- net GND: track 1.27 -> 61.7 mm, vias 70 -> 106
- net /USB PD Charger/VBUS: track 1.41 -> 49.8 mm, vias 1 -> 2
- net /USB PD Charger/CC: track 1.41 -> 44.5 mm, vias 1 -> 2
- net Net-(J11-Pin_2): track 75.3 -> 62.0 mm
- net Net-(J11-Pin_6): track 41.2 -> 34.0 mm
- net /USB C DFPs/USB_DFP0_VBUS: track 56.2 -> 62.3 mm, vias 5 -> 3
- net Net-(JP7-A): track 39.9 -> 45.2 mm
- net /USB C DFPs/USB_DFP1_VBUS: track 33.6 -> 32.8 mm, vias 5 -> 2
- net /C_RXP: track 35.4 -> 34.7 mm
- net /C_RXN: track 35.4 -> 34.6 mm
- net +3V3: track 531.4 -> 531.1 mm, vias 48 -> 47
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Other:
- board size 174.7 x 76.7 mm -> 166.2 x 80.5 mm
- board text added: "AC_L"
- board text added: "CC"
- board text added: "C_DET"
- board text added: "DET1"
- board text added: "DET2"
- board text added: "IRQ#"
- board text added: "Option A: ATX Power"
- board text added: "Option B: XG Station Power"
- board text added: "PEN"
- board text added: "POK"
- board text added: "RST"
- board text added: "RSV0"
- board text added: "SCLK"
- board text added: "SDAT"
- board text added: "VBUS"
- board text added: "XG Mobile Dock v0.1"
- board text removed: "${REFERENCE}"
