File: XG_Mobile_Dock_Lite.kicad_pcb (KiCad board)
At the start: 4 copper layers, 220 x 65 mm, 60 parts, among them J1 5-1775443-8, J10 SWD, J11 UART, J12 I2C1, J13 39300240, J14 469911008, J17 8730, J2 20455-040E-76, J3 20455-040E-76, J4 3-2362375-4, J5 USB_C_Receptacle, Q16 AO3401A, Q17 2N7002W, SW1 SW_Push, U1 AMS1117-3.3, U12 STM32F030C8Tx

Commit message: pcb: fix +3.3V rail for cable LED
Connections:
- J3 pad 1: /+3V3_PCI -> +3V3
- J3 pad 2: /+3V3_PCI -> +3V3
- J3 pad 3: /+3V3_PCI -> +3V3
- J3 pad 4: /+3V3_PCI -> +3V3
Routing:
- net /+3V3_PCI: track 84.4 -> 0.00 mm, vias 18 -> 12
- net +3V3: vias 14 -> 20
Changed lines of the file:
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@@
 			(size 0.25 0.9)
 			(layers "F.Cu" "F.Mask" "F.Paste")
-			(net 173 "/+3V3_PCI")
+			(net 2 "+3V3")
 			(pinfunction "+3.3V")
 			(pintype "passive")
@@
 			(size 0.25 0.9)
 			(layers "F.Cu" "F.Mask" "F.Paste")
-			(net 173 "/+3V3_PCI")
+			(net 2 "+3V3")
 			(pinfunction "+3.3V")
 			(pintype "passive")
@@
 			(size 0.25 0.9)
 			(layers "F.Cu" "F.Mask" "F.Paste")
-			(net 173 "/+3V3_PCI")
+			(net 2 "+3V3")
 			(pinfunction "+3.3V")
 			(pintype "passive")
@@
 			(size 0.25 0.9)
 			(layers "F.Cu" "F.Mask" "F.Paste")
-			(net 173 "/+3V3_PCI")
+			(net 2 "+3V3")
 			(pinfunction "+3.3V")
 			(pintype "passive")
@@
 	)
 	(via
+		(at 148.121496 85.171496)
+		(size 0.5)
+		(drill 0.3)
+		(layers "F.Cu" "B.Cu")
+		(free yes)
+		(net 2)
+	)
+	(via
 		(at 177.75 43.25)
 		(size 0.5)
@@
 	)
 	(via
+		(at 148.121496 84.371496)
+		(size 0.5)
+		(drill 0.3)
+		(layers "F.Cu" "B.Cu")
+		(free yes)
+		(net 2)
+	)
+	(via
 		(at 175.5 42.5)
 		(size 0.5)
@@
 	)
 	(via
+		(at 148.121496 85.971496)
+		(size 0.5)
+		(drill 0.3)
+		(layers "F.Cu" "B.Cu")
+		(free yes)
+		(net 2)
+	)
+	(via
 		(at 168.862597 81.121496)
 		(size 0.5)
@@
 	)
 	(via
+		(at 147.121496 85.971496)
+		(size 0.5)
+		(drill 0.3)
+		(layers "F.Cu" "B.Cu")
+		(free yes)
+		(net 2)
+	)
+	(via
 		(at 178.5 42.5)
 		(size 0.5)
@@
 	)
 	(via
+		(at 147.121496 84.371496)
+		(size 0.5)
+		(drill 0.3)
+		(layers "F.Cu" "B.Cu")
+		(free yes)
+		(net 2)
+	)
+	(via
 		(at 177 44)
 		(size 0.5)
@@
 	)
 	(via
+		(at 147.121496 85.171496)
+		(size 0.5)
+		(drill 0.3)
+		(layers "F.Cu" "B.Cu")
+		(free yes)
+		(net 2)
+	)
+	(via
 		(at 168.862597 83.621496)
 		(size 0.5)
@@
 	)
 	(via
-		(at 148.121496 85.171496)
-		(size 0.5)
-		(drill 0.3)
-		(layers "F.Cu" "B.Cu")
-		(free yes)
-		(net 173)
-	)
-	(via
 		(at 85.83666 59.279018)
 		(size 0.5)
@@
 	)
 	(via
-		(at 148.121496 84.371496)
-		(size 0.5)
-		(drill 0.3)
-		(layers "F.Cu" "B.Cu")
-		(free yes)
-		(net 173)
-	)
-	(via
 		(at 85.83666 61.029018)
 		(size 0.5)
@@
 	)
 	(via
-		(at 148.121496 85.971496)
-		(size 0.5)
-		(drill 0.3)
-		(layers "F.Cu" "B.Cu")
-		(free yes)
-		(net 173)
-	)
-	(via
 		(at 84.83666 61.029018)
 		(size 0.5)
@@
 	)
 	(via
-		(at 147.121496 85.971496)
-		(size 0.5)
-		(drill 0.3)
-		(layers "F.Cu" "B.Cu")
-		(free yes)
-		(net 173)
-	)
-	(via
 		(at 86.83666 62.029018)
 		(size 0.5)
@@
 	)
 	(via
-		(at 147.121496 84.371496)
-		(size 0.5)
-		(drill 0.3)
-		(layers "F.Cu" "B.Cu")
-		(free yes)
-		(net 173)
-	)
-	(via
 		(at 86.83666 59.279018)
 		(size 0.5)
@@
 	)
 	(via
-		(at 147.121496 85.171496)
-		(size 0.5)
-		(drill 0.3)
-		(layers "F.Cu" "B.Cu")
-		(free yes)
-		(net 173)
-	)
-	(via
 		(at 85.83666 58.279018)
 		(size 0.5)
@@
 		(net 173)
 	)
-	(segment
-		(start 147.5 88.25)
-		(end 147.5 87.5)
-		(width 1.5)
-		(layer "In1.Cu")
-		(net 173)
-	)
-	(segment
-		(start 84.917496 72.758603)
-		(end 84.917496 63.377496)
-		(width 1.5)
-		(layer "In1.Cu")
-		(net 173)
-	)
-	(segment
-		(start 143.496514 92.154)
-		(end 143.596 92.154)
-		(width 1.5)
-		(layer "In1.Cu")
-		(net 173)
-	)
-	(segment
-		(start 146.5 89.25)
-		(end 147.5 88.25)
-		(width 1.5)
-		(layer "In1.Cu")
-		(net 173)
-	)
-	(segment
-		(start 143.596 92.154)
-		(end 146.5 89.25)
-		(width 1.5)
-		(layer "In1.Cu")
-		(net 173)
-	)
-	(segment
-		(start 143.496514 92.154)
-		(end 104.312893 92.154)
-		(width 1.5)
-		(layer "In1.Cu")
-		(net 173)
-	)
-	(segment
-		(start 104.312893 92.154)
-		(end 84.917496 72.758603)
-		(width 1.5)
-		(layer "In1.Cu")
-		(net 173)
-	)
-	(segment
-		(start 84.917496 63.377496)
-		(end 86.917496 63.377496)
-		(width 1.5)
-		(layer "In1.Cu")
-		(net 173)
-	)
 	(zone
 		(net 118)
@@
 	)
 	(zone
+		(net 2)
+		(net_name "+3V3")
+		(layer "F.Cu")
+		(hatch edge 0.5)
+		(priority 21)
+		(connect_pads yes
+			(clearance 0)
+		)
+		(min_thickness 0.25)
+		(filled_areas_thickness no)
+		(fill yes
+			(thermal_gap 0.5)
+			(thermal_bridge_width 0.5)
+		)
+		(polygon
+			(pts
+				(xy 148.621496 87.621496) (xy 146.621496 87.621496) (xy 146.621496 83.871496) (xy 148.621496 83.871496)
+			)
+		)
+	)
+	(zone
 		(net 1)
 		(net_name "GND")
@@
 	)
 	(zone
-		(net 173)
-		(net_name "/+3V3_PCI")
-		(layers "F.Cu" "In1.Cu")
+		(net 2)
+		(net_name "+3V3")
+		(layer "In1.Cu")
 		(hatch edge 0.5)
-		(priority 21)
+		(priority 9)
 		(connect_pads yes
 			(clearance 0)
@@
 		(polygon
 			(pts
-				(xy 148.621496 87.621496) (xy 146.621496 87.621496) (xy 146.621496 83.871496) (xy 148.621496 83.871496)
+				(xy 175 44.5) (xy 175 39.5) (xy 185.121496 39.529018) (xy 185.121496 44.5)
 			)
 		)
@@
 		(layer "In1.Cu")
 		(hatch edge 0.5)
-		(priority 9)
+		(priority 21)
 		(connect_pads yes
 			(clearance 0)
@@
 		(polygon
 			(pts
-				(xy 175 44.5) (xy 175 39.5) (xy 185.121496 39.529018) (xy 185.121496 44.5)
+				(xy 168.621496 87.621496) (xy 146.621496 87.621496) (xy 146.621496 83.871496) (xy 168.621496 83.871496)
 			)
 		)
@@
 		(polygon
 			(pts
-				(xy 88.871496 54.621496) (xy 88.871496 92.121496) (xy 135.621496 92.121496) (xy 135.621496 54.621496)
+				(xy 88.871496 54.621496) (xy 88.871496 92.121496) (xy 139.121496 92.121496) (xy 139.121496 54.621496)
 			)
 		)
